File: KiCad/CustomTemperatureController.kicad_pcb (KiCad board)
At the start: 2 copper layers, 62 x 94 mm, 77 parts, among them J1 USB_C, J10 Aux, J2 AUX1, J3 AUX2, J7 UART, J8 I2C, J9 I2C, K1 SANYOU_SRD-05VDC, K2 SANYOU_SRD-05VDC, Q1 SS8050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

Commit message: Rev101 add resistors.
Parts:
- removed 3V3: 3V3_TP, TestPoint:TestPoint_Pad_D1.0mm
- removed 5V: 5V_TP, TestPoint:TestPoint_Pad_D1.0mm
- removed GND: GND_TP, TestPoint:TestPoint_Pad_D1.0mm
- removed L: AC_IN, Connector_Wire:SolderWire-1.5sqmm_1x02_P6mm_D1.7mm_OD3mm
- removed L1: L1_OUT, Connector_Wire:SolderWire-1.5sqmm_1x01_D1.7mm_OD3mm
- removed L2: L2_OUT, Connector_Wire:SolderWire-1.5sqmm_1x01_D1.7mm_OD3mm
- removed N: N_OUT, Connector_Wire:SolderWire-1.5sqmm_1x01_D1.7mm_OD3mm
- removed OW: ONEWIRE_TP, TestPoint:TestPoint_Pad_D1.0mm
- removed RST: RST_TP, TestPoint:TestPoint_Pad_D1.0mm
- added R20: 22k, Resistor_SMD:R_0805_2012Metric, F.Cu at (123.1, 64.1)
- added R21: 47k, Resistor_SMD:R_0805_2012Metric, F.Cu at (121.2, 64.1)
- moved TP9 4.34 mm to (126.7, 63.2)
- moved R13 0.69 mm to (130.2, 63.1)
Connections:
- U3 pad 8: /V_BUS -> Net-(U3-VBUS)
Routing:
- net /V_BUS: track 39.9 -> 35.9 mm
- net Net-(U3-VBUS): track 0.00 -> 3.44 mm
- net GND: track 125.6 -> 124.5 mm
- net Net-(J1-SHIELD): track 21.2 -> 20.7 mm

Commit message: Update revision text on board.
Other:
- board text added: "28/01/2025 v1.0.1"
- board text removed: "28/01/2025 v1.0"
Changed lines of the file:
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@@
 		)
 	)
-	(gr_text "28/01/2025 v1.0"
+	(gr_text "28/01/2025 v1.0.1"
 		(at 120 60.25 0)
 		(layer "F.SilkS")
